Commit message: minor changes to gazebo system robot still not moving

File: ws/src/car_description/urdf/gazebo_control.xacro (robot description, xacro)
@@ -2,10 +2,6 @@
   <gazebo>
     <plugin
-      filename="libros_gz_control.so"
-      name="ros_gz_control::GazeboSystem">
-      <ros>
-        <namespace>/</namespace>
-      </ros>
-    </plugin>
+      filename="libgz_ros2_control-system.so"
+      name="gz_ros2_control::GazeboSystem"/>
   </gazebo>
 </robot>

File: ws/src/car_description/urdf/wheels.xacro (robot description, xacro)
@@ -1,110 +1,144 @@
 <?xml version="1.0"?>
 <robot xmlns:xacro="http://www.ros.org/wiki/xacro">
-    <!-- =========================================================
-         Local includes (each file must be self-contained)
-         ========================================================= -->
-    <xacro:include filename="inertial_macros.xacro"/>
-    <!-- <xacro:include filename="materials.xacro"/> -->
-    <!-- =========================================================
-         Constants (avoid cross-file dependencies)
-         ========================================================= -->
-    <!-- -90 degrees in radians -->
-    <xacro:property name="wheel_rpy_x" value="-1.57079632679"/>
-    <!-- =========================================================
-         FRONT WHEELS (fixed to steering links)
-         ========================================================= -->
-    <!-- Front Left Wheel -->
-    <joint name="front_left_wheel_joint" type="fixed">
-        <parent link="front_left_steering_link"/>
-        <child link="front_left_wheel"/>
-        <origin xyz="0 0 0" rpy="${wheel_rpy_x} 0 0"/>
-    </joint>
-    <link name="front_left_wheel">
-        <visual>
-            <geometry>
-                <cylinder radius="0.05" length="0.04"/>
-            </geometry>
-            <material name="blue"/>
-        </visual>
-        <collision>
-            <geometry>
-                <cylinder radius="0.05" length="0.04"/>
-            </geometry>
-        </collision>
-        <!-- IMPORTANT: inertial_cylinder REQUIRES an <origin> block -->
-        <xacro:inertial_cylinder mass="0.1" radius="0.05" length="0.04">
-            <origin xyz="0 0 0" rpy="0 0 0"/>
-        </xacro:inertial_cylinder>
-    </link>
-    <!-- Front Right Wheel -->
-    <joint name="front_right_wheel_joint" type="fixed">
-        <parent link="front_right_steering_link"/>
-        <child link="front_right_wheel"/>
-        <origin xyz="0 0 0" rpy="${wheel_rpy_x} 0 0"/>
-    </joint>
-    <link name="front_right_wheel">
-        <visual>
-            <geometry>
-                <cylinder radius="0.05" length="0.04"/>
-            </geometry>
-            <material name="blue"/>
-        </visual>
-        <collision>
-            <geometry>
-                <cylinder radius="0.05" length="0.04"/>
-            </geometry>
-        </collision>
-        <xacro:inertial_cylinder mass="0.1" radius="0.05" length="0.04">
-            <origin xyz="0 0 0" rpy="0 0 0"/>
-        </xacro:inertial_cylinder>
-    </link>
-    <!-- =========================================================
-         REAR WHEELS (driven, continuous joints)
-         ========================================================= -->
-    <!-- Rear Left Wheel -->
-    <joint name="rear_left_wheel_joint" type="continuous">
-        <parent link="base_link"/>
-        <child link="rear_left_wheel"/>
-        <origin xyz="-0.15 0.175 0" rpy="${wheel_rpy_x} 0 0"/>
-        <axis xyz="0 0 1"/>
-    </joint>
-    <link name="rear_left_wheel">
-        <visual>
-            <geometry>
-                <cylinder radius="0.05" length="0.04"/>
-            </geometry>
-            <material name="blue"/>
-        </visual>
-        <collision>
-            <geometry>
-                <cylinder radius="0.05" length="0.04"/>
-            </geometry>
-        </collision>
-        <xacro:inertial_cylinder mass="0.1" radius="0.05" length="0.04">
-            <origin xyz="0 0 0" rpy="0 0 0"/>
-        </xacro:inertial_cylinder>
-    </link>
-    <!-- Rear Right Wheel -->
-    <joint name="rear_right_wheel_joint" type="continuous">
-        <parent link="base_link"/>
-        <child link="rear_right_wheel"/>
-        <origin xyz="-0.15 -0.175 0" rpy="${wheel_rpy_x} 0 0"/>
-        <axis xyz="0 0 1"/>
-    </joint>
-    <link name="rear_right_wheel">
-        <visual>
-            <geometry>
-                <cylinder radius="0.05" length="0.04"/>
-            </geometry>
-            <material name="blue"/>
-        </visual>
-        <collision>
-            <geometry>
-                <cylinder radius="0.05" length="0.04"/>
-            </geometry>
-        </collision>
-        <xacro:inertial_cylinder mass="0.1" radius="0.05" length="0.04">
-            <origin xyz="0 0 0" rpy="0 0 0"/>
-        </xacro:inertial_cylinder>
-    </link>
+  <!-- =========================================================
+       Properties
+       ========================================================= -->
+  <!-- Rotate wheels so cylinder axis aligns with rolling direction -->
+  <!-- =========================================================
+       FRONT WHEELS (fixed to steering links)
+       ========================================================= -->
+  <!-- Front Left Wheel -->
+  <joint name="front_left_wheel_joint" type="fixed">
+    <parent link="front_left_steering_link"/>
+    <child link="front_left_wheel"/>
+    <origin xyz="0 0 0" rpy="-1.5708 0 0"/>
+  </joint>
+  <link name="front_left_wheel">
+    <visual>
+      <geometry>
+        <cylinder radius="0.05" length="0.04"/>
+      </geometry>
+    </visual>
+    <collision>
+      <origin xyz="0 0 -0.05"/>
+      <geometry>
+        <cylinder radius="0.05" length="0.04"/>
+      </geometry>
+    </collision>
+    <inertial>
+      <origin xyz="0 0 0"/>
+      <mass value="0.5"/>
+      <inertia ixx="0.001" iyy="0.001" izz="0.001"
+               ixy="0.0" ixz="0.0" iyz="0.0"/>
+    </inertial>
+  </link>
+  <!-- Front Right Wheel -->
+  <joint name="front_right_wheel_joint" type="fixed">
+    <parent link="front_right_steering_link"/>
+    <child link="front_right_wheel"/>
+    <origin xyz="0 0 0" rpy="-1.5708 0 0"/>
+  </joint>
+  <link name="front_right_wheel">
+    <visual>
+      <geometry>
+        <cylinder radius="0.05" length="0.04"/>
+      </geometry>
+    </visual>
+    <collision>
+      <origin xyz="0 0 -0.05"/>
+      <geometry>
+        <cylinder radius="0.05" length="0.04"/>
+      </geometry>
+    </collision>
+    <inertial>
+      <origin xyz="0 0 0"/>
+      <mass value="0.5"/>
+      <inertia ixx="0.001" iyy="0.001" izz="0.001"
+               ixy="0.0" ixz="0.0" iyz="0.0"/>
+    </inertial>
+  </link>
+  <!-- =========================================================
+       REAR WHEELS (DRIVEN)
+       ========================================================= -->
+  <!-- Rear Left Wheel -->
+  <joint name="rear_left_wheel_joint" type="continuous">
+    <parent link="base_link"/>
+    <child link="rear_left_wheel"/>
+    <origin xyz="-0.15 0.175 0" rpy="-1.5708 0 0"/>
+    <!-- CRITICAL FIX: correct rolling axis -->
+    <axis xyz="0 1 0"/>
+  </joint>
+  <link name="rear_left_wheel">
+    <visual>
+      <geometry>
+        <cylinder radius="0.05" length="0.04"/>
+      </geometry>
+    </visual>
+    <collision>
+      <origin xyz="0 0 -0.05"/>
+      <geometry>
+        <cylinder radius="0.05" length="0.04"/>
+      </geometry>
+    </collision>
+    <inertial>
+      <origin xyz="0 0 0"/>
+      <mass value="0.5"/>
+      <inertia ixx="0.001" iyy="0.001" izz="0.001"
+               ixy="0.0" ixz="0.0" iyz="0.0"/>
+    </inertial>
+  </link>
+  <!-- Rear Right Wheel -->
+  <joint name="rear_right_wheel_joint" type="continuous">
+    <parent link="base_link"/>
+    <child link="rear_right_wheel"/>
+    <origin xyz="-0.15 -0.175 0" rrpy="-1.5708 0 0"/>
+    <!-- CRITICAL FIX: correct rolling axis -->
+    <axis xyz="0 1 0"/>
+  </joint>
+  <link name="rear_right_wheel">
+    <visual>
+      <geometry>
+        <cylinder radius="0.05" length="0.04"/>
+      </geometry>
+    </visual>
+    <collision>
+      <origin xyz="0 0 -0.05"/>
+      <geometry>
+        <cylinder radius="0.05" length="0.04"/>
+      </geometry>
+    </collision>
+    <inertial>
+      <origin xyz="0 0 0"/>
+      <mass value="0.5"/>
+      <inertia ixx="0.001" iyy="0.001" izz="0.001"
+               ixy="0.0" ixz="0.0" iyz="0.0"/>
+    </inertial>
+  </link>
+  <!-- =========================================================
+       Gazebo Friction (MANDATORY)
+       ========================================================= -->
+  <gazebo reference="front_left_wheel">
+    <mu1>1.2</mu1>
+    <mu2>1.2</mu2>
+    <kp>100000.0</kp>
+    <kd>10.0</kd>
+  </gazebo>
+  <gazebo reference="front_right_wheel">
+    <mu1>1.2</mu1>
+    <mu2>1.2</mu2>
+    <kp>100000.0</kp>
+    <kd>10.0</kd>
+  </gazebo>
+  <gazebo reference="rear_left_wheel">
+    <mu1>1.2</mu1>
+    <mu2>1.2</mu2>
+    <kp>100000.0</kp>
+    <kd>10.0</kd>
+  </gazebo>
+  <gazebo reference="rear_right_wheel">
+    <mu1>1.2</mu1>
+    <mu2>1.2</mu2>
+    <kp>100000.0</kp>
+    <kd>10.0</kd>
+  </gazebo>
 </robot>

Commit message: some fixes let me fix this again

File: ws/src/car_description/urdf/gazebo_control.xacro (robot description, xacro)
@@ -2,6 +2,10 @@
   <gazebo>
     <plugin
-      filename="libgz_ros2_control-system.so"
-      name="gz_ros2_control::GazeboSystem"/>
+      filename="libros_gz_sim_ros2_control.so"
+      name="ros_gz_sim::RosGzSimRos2ControlPlugin">
+      <ros>
+        <namespace>/</namespace>
+      </ros>
+    </plugin>
   </gazebo>
 </robot>

File: ws/src/car_description/urdf/ros2_control.xacro (robot description, xacro)
@@ -2,7 +2,7 @@
 <robot xmlns:xacro="http://www.ros.org/wiki/xacro">
     <ros2_control name="NavStackSystem" type="system">
-          <hardware>
-            <plugin>gz_ros2_control/GazeboSystem</plugin>
-          </hardware>
+        <hardware>
+            <type>system</type>
+        </hardware>
         <joint name="front_left_steering_joint">
             <command_interface name="position"/>

File: ws/src/car_description/urdf/wheels.xacro (robot description, xacro)
@@ -92,5 +92,5 @@
     <parent link="base_link"/>
     <child link="rear_right_wheel"/>
-    <origin xyz="-0.15 -0.175 0" rrpy="-1.5708 0 0"/>
+    <origin xyz="-0.15 -0.175 0" rpy="-1.5708 0 0"/>
     <!-- CRITICAL FIX: correct rolling axis -->
     <axis xyz="0 1 0"/>
